Commit message: add gazebo model and plugins of each sensor

File: jackal_description/urdf/accessories.urdf.xacro (robot description, xacro)
@@ -461,3 +461,23 @@
     </gazebo>
   </xacro:if>
+  <!-- Create virtual URDF and corresponding plugins for the Gazebo -->
+  <xacro:if value="${use_gazebo}">
+    <!-- Intel Realsense D435 Camera -->
+    <xacro:include filename="$(find jackal_description)/urdf/accessories/realsense_d435.urdf.xacro" />
+    <xacro:D435 name="virtual_camera" topics_ns="camera" parent="camera_link" publish_pointcloud="true">
+      <origin xyz="-0.015 0 -0.0125" rpy="0 0 0" />
+    </xacro:D435>
+    <!-- SICK TIM571 2D LiDAR -->
+    <xacro:include filename="$(find sick_scan)/urdf/sick_scan.urdf.xacro" />
+    <joint name="virtual_tim571_mount_joint" type="fixed">
+      <parent link="tim571" />
+      <child link="virtual_tim571_mount_link" />
+      <origin rpy="0 0 0" xyz="0 0 -0.01665"/>
+    </joint>
+    <xacro:sick_tim_57x name="virtual_tim571" ros_topic="sick_scan" />
+    <!-- Velodyne VLP-16 (Puck) 3D LiDAR -->
+    <xacro:VLP-16 parent="velodyne" name="virtual_velodyne" topic="velodyne_scan" organize_cloud="true" gpu="true">
+      <origin xyz="0 0 0" rpy="0 0 0.02" />
+    </xacro:VLP-16>
+  </xacro:if>
 </robot>

File: jackal_description/urdf/jackal.urdf.xacro (robot description, xacro)
@@ -13,4 +13,6 @@
   <xacro:property name="dummy_inertia" value="1e-09"/>
   <xacro:property name="mount_spacing" value="0.120" />
+  <xacro:arg name="gazebo" default="true" />
+  <xacro:property name="use_gazebo" value="$(arg gazebo)" />
   <material name="dark_grey"><color rgba="0.2 0.2 0.2 1.0" /></material>
   <material name="light_grey"><color rgba="0.4 0.4 0.4 1.0" /></material>
