Commit message: add custom mounts

File: jackal_description/urdf/jackal.urdf.xacro (robot description, xacro)
@@ -228,3 +228,44 @@
   <!-- Optional for Clearpath internal softwares -->
   <xacro:include filename="$(optenv CPR_URDF_EXTRAS empty.urdf)" />
+  <!-- ROAS TOP -->
+  <link name="top_structure">
+    <visual>
+      <origin xyz="0 0 0" rpy="0 0 0"/>
+      <geometry>
+        <mesh filename="package://jackal_description/meshes/A-PSI-23-0313-01_A0001.STL"/>
+      </geometry>
+      <material name="silver">
+        <color rgba="0.75 0.75 0.75 1"/>
+      </material>
+    </visual>
+    <collision>
+      <origin xyz="0 0 0" rpy="0 0 0"/>
+      <geometry>
+        <mesh filename="package://jackal_description/meshes/A-PSI-23-0313-01_A0001.STL"/>
+      </geometry>
+    </collision>
+  </link>
+  <joint name="top_structure_joint" type="fixed">
+    <parent link="base_link"/>
+    <child link="top_structure"/>
+    <origin xyz="0 0 -0.0690" rpy="0 0 0"/>
+  </joint>
+<link name="camera_link"/>
+<joint name="camera_joint" type="fixed">
+    <parent link="top_structure"/>
+    <child link="camera_link"/>
+    <origin xyz="0.28165 0 0.1461" rpy="0 0 0"/>
+</joint>
+<link name="tim571"/>
+<joint name="Tim571_joint" type="fixed">
+    <parent link="top_structure"/>
+    <child link="tim571"/>
+    <origin xyz="0.169 0 0.28356" rpy="0 0 0"/>
+</joint>
+<link name="velodyne"/>
+<joint name="Velodyne_joint" type="fixed">
+    <parent link="top_structure"/>
+    <child link="velodyne"/>
+    <origin xyz="0.050 0 0.3575" rpy="0 0 0"/>
+</joint>
 </robot>

Commit message: paint the accessories

File: jackal_description/urdf/jackal.urdf.xacro (robot description, xacro)
@@ -233,5 +233,5 @@
       <origin xyz="0 0 0" rpy="0 0 0"/>
       <geometry>
-        <mesh filename="package://jackal_description/meshes/A-PSI-23-0313-01_A0001.STL"/>
+        <mesh filename="package://jackal_description/meshes/A-PSI-23-0313-01_A0001.obj"/>
       </geometry>
       <material name="silver">
@@ -242,5 +242,5 @@
       <origin xyz="0 0 0" rpy="0 0 0"/>
       <geometry>
-        <mesh filename="package://jackal_description/meshes/A-PSI-23-0313-01_A0001.STL"/>
+        <mesh filename="package://jackal_description/meshes/A-PSI-23-0313-01_A0001.obj"/>
       </geometry>
     </collision>

Commit message: add options for gpu

File: jackal_description/urdf/jackal.urdf.xacro (robot description, xacro)
@@ -14,5 +14,7 @@
   <xacro:property name="mount_spacing" value="0.120" />
   <xacro:arg name="gazebo" default="true" />
+  <xacro:arg name="gpu" default="true" />
   <xacro:property name="use_gazebo" value="$(arg gazebo)" />
+  <xacro:property name="use_gpu" value="$(arg gpu)" />
   <material name="dark_grey"><color rgba="0.2 0.2 0.2 1.0" /></material>
   <material name="light_grey"><color rgba="0.4 0.4 0.4 1.0" /></material>
